File: PRJ4/PRJ4 (Alimentador Digital)/PRJ4 (Alimentador Digital).kicad_sch (KiCad schematic)
At the start: 48 parts, among them J1 Load Cell, J2 DC_MOTOR, J4 Conn_01x04, J5 Conn_01x02, J6 Conn_01x07, SW1 SW_Push, SW2 SW_SPDT, SW3 SW_SPDT, SW4 BT4, SW5 BT3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

Commit message: att da pcb v2
Parts:
- removed SW4: BT4, Button_Switch_SMD:SW_SPST_B3U-1000P-B, symbol Switch:SW_Push
- removed SW5: BT3, Button_Switch_SMD:SW_SPST_B3U-1000P-B, symbol Switch:SW_Push
- removed SW6: BT2, Button_Switch_SMD:SW_SPST_B3U-1000P-B, symbol Switch:SW_Push
- removed SW7: BT1, Button_Switch_SMD:SW_SPST_B3U-1000P-B, symbol Switch:SW_Push
- added H1, H2, H3, H4: MountingHole, MountingHole:MountingHole_3.2mm_M3, symbol Mechanical:MountingHole
Connections:
- net CLK__DSP: now also U1.55 (PB3); no longer U1.57 (PB5)
- net MOSI_DSP: now also U1.57 (PB5); no longer U1.55 (PB3)
- net BT1: no longer names the net of U1.51 (PC10)
- net BT2: no longer names the net of U1.52 (PC11)
- net BT3: no longer names the net of U1.53 (PC12)
- net BT4: no longer names the net of U1.50 (PA15)
- no-connect marks 44 -> 48
Other:
- note removed: "Buttons"
- moved on the sheet: C10, C11, C12, C13, C14, C15, C16, C17, C9, FB1

Commit message: nomes do pinos
Connections:
- net CLK__DSP renamed SCL_DSP
- net MOSI_DSP renamed SDA_DSP
- net RES_DSP renamed RESET_DSP
Changed lines of the file:
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@@
 		)
 	)
-	(label "RES_DSP"
+	(label "RESET_DSP"
 		(at 139.7 50.8 0)
 		(fields_autoplaced yes)
@@
 		)
 	)
-	(label "MOSI_DSP"
-		(at 168.91 34.29 180)
-		(fields_autoplaced yes)
-		(effects
-			(font
-				(size 1.27 1.27)
-			)
-			(justify right bottom)
-		)
-	)
 	(label "LOAD_OUT"
 		(at 101.6 66.04 180)
@@
 		)
 	)
-	(label "CLK__DSP"
-		(at 168.91 31.75 180)
-		(fields_autoplaced yes)
-		(effects
-			(font
-				(size 1.27 1.27)
-			)
-			(justify right bottom)
-		)
-	)
 	(label "DC1_IN2"
 		(at 34.29 176.53 180)
@@
 		)
 	)
+	(label "SDA_DSP"
+		(at 168.91 34.29 180)
+		(fields_autoplaced yes)
+		(effects
+			(font
+				(size 1.27 1.27)
+			)
+			(justify right bottom)
+		)
+	)
 	(label "VDDA"
 		(at 217.17 27.94 90)
@@
 		)
 	)
-	(label "MOSI_DSP"
+	(label "SDA_DSP"
 		(at 139.7 96.52 0)
 		(fields_autoplaced yes)
@@
 		)
 	)
-	(label "RES_DSP"
+	(label "RESET_DSP"
 		(at 168.91 36.83 180)
 		(fields_autoplaced yes)
@@
 		)
 	)
-	(label "CLK__DSP"
+	(label "SCL_DSP"
+		(at 168.91 31.75 180)
+		(fields_autoplaced yes)
+		(effects
+			(font
+				(size 1.27 1.27)
+			)
+			(justify right bottom)
+		)
+	)
+	(label "SCL_DSP"
 		(at 139.7 91.44 0)
 		(fields_autoplaced yes)
