File: PRJ4/PRJ4 (Alimentador Digital)/PRJ4 (Alimentador Digital).kicad_pcb (KiCad board)
At the start: 4 copper layers, 55.2 x 62.9 mm, 53 parts, among them J1 Load Cell, J2 DC_MOTOR, J4 Conn_01x04, J5 Conn_01x02, J6 Conn_01x07, SW1 SW_Push, SW2 SW_SPDT, SW3 SW_SPDT, SW4 BT4, SW5 BT3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

Commit message: att da pcb v2
Parts:
- removed SW4: BT4, Button_Switch_SMD:SW_SPST_B3U-1000P-B
- removed SW5: BT3, Button_Switch_SMD:SW_SPST_B3U-1000P-B
- removed SW6: BT2, Button_Switch_SMD:SW_SPST_B3U-1000P-B
- removed SW7: BT1, Button_Switch_SMD:SW_SPST_B3U-1000P-B
- H1, H2, H3, H4: value MountingHole_3.2mm_M3 -> MountingHole
- moved J5 6.79 mm to (167.8, 111.7)
- moved J6 5.44 mm to (168.0, 103.4)
- moved J2 4.60 mm to (168.0, 82.2)
Connections:
- U1 pad 50: /BT4 -> unconnected-(U1-PA15-Pad50)
- U1 pad 51: /BT1 -> unconnected-(U1-PC10-Pad51)
- U1 pad 52: /BT2 -> unconnected-(U1-PC11-Pad52)
- U1 pad 53: /BT3 -> unconnected-(U1-PC12-Pad53)
- U1 pad 55: /MOSI_DSP -> /CLK__DSP
- U1 pad 57: /CLK__DSP -> /MOSI_DSP
Routing:
- net +3.3V: track 231.7 -> 205.4 mm, vias 8 -> 5
- net /BT3: track 12.5 -> 0.00 mm
- net /BT4: track 8.10 -> 0.00 mm
- net /BT2: track 7.83 -> 0.00 mm
- net /BT1: track 5.45 -> 0.00 mm
- net GND: track 11.0 -> 15.7 mm, vias 68 -> 80
- net +9V: track 69.0 -> 73.0 mm
- net Net-(J2-Pin_2): track 4.89 -> 8.56 mm
- net /CLK__DSP: track 41.0 -> 43.9 mm
- net Net-(J2-Pin_1): track 4.38 -> 7.32 mm
- net /DC_DSP: track 33.6 -> 31.4 mm
- net /RES_DSP: track 35.3 -> 33.2 mm
- net /MOSI_DSP: track 39.1 -> 37.6 mm
- net /BLK_DSP: track 31.8 -> 30.8 mm

Commit message: mudei os pinos
Connections:
- net /CLK__DSP renamed /SCL_DSP
- net /MOSI_DSP renamed /SDA_DSP
- net /RES_DSP renamed /RESET_DSP
